Commit message: made gz's to new package

File: core_gz/urdf/core2025_attacker.urdf (robot description, URDF)
Before this commit: robot core2025_attacker, 5 links, 4 joints
Links:
- link base_link: geometry collision mesh filename=package://core_gz/urdf/mesh/Attacker_Shooter.dae; visual mesh filename=package://core_gz/urdf/mesh/Attacker_Shooter.dae
- link chassis_link: geometry collision mesh filename=package://core_gz/urdf/mesh/Attacker_Chassis.dae; visual mesh filename=package://core_gz/urdf/mesh/Attacker_Chassis.dae
- link upperwing_link: geometry collision mesh filename=package://core_gz/urdf/mesh/Attacker_UpperWing.dae; visual mesh filename=package://core_gz/urdf/mesh/Attacker_UpperWing.dae
