Commit message: Refactor code structure for improved readability and maintainability

File: core_launch/urdf/core2025_attacker.urdf (robot description, URDF)
Before this commit: robot core2025_attacker, 5 links, 4 joints
Links:
- link base_link: geometry collision mesh filename=package://core_launch/urdf/mesh/attacker_shooter.dae; visual mesh filename=package://core_launch/urdf/mesh/attacker_shooter.dae
- link chassis_link: geometry collision mesh filename=package://core_launch/urdf/mesh/attacker_chassis.dae; visual mesh filename=package://core_launch/urdf/mesh/attacker_chassis.dae
- link upperwing_link: geometry collision mesh filename=package://core_launch/urdf/mesh/attacker_upperwing.dae; visual mesh filename=package://core_launch/urdf/mesh/attacker_upperwing.dae
